Commit message: nothing

File: urdf/yieldbotvf.xacro (robot description, xacro)
@@ -27,4 +27,18 @@
   </collision>
 </link>
+<link name="base_footprint">
+  <visual>
+    <origin xyz="0 0 0" rpy="0 0 0"/>
+    <geometry>
+      <box size="0.01 0.01 0.01"/>  <!-- Optionally, you can define a small box -->
+    </geometry>
+    <material name="blue"/>
+  </visual>
+</link>
+<joint name="base_link_to_base_footprint" type="fixed">
+  <origin xyz="0 0 0" rpy="0 0 0"/>
+  <parent link="base_link"/>
+  <child link="base_footprint"/>
+</joint>
 <link name="roue_avd_1">
   <inertial>

Commit message: base footprint

File: urdf/yieldbotvf.xacro (robot description, xacro)
@@ -27,18 +27,4 @@
   </collision>
 </link>
-<link name="base_footprint">
-  <visual>
-    <origin xyz="0 0 0" rpy="0 0 0"/>
-    <geometry>
-      <box size="0.01 0.01 0.01"/>  <!-- Optionally, you can define a small box -->
-    </geometry>
-    <material name="blue"/>
-  </visual>
-</link>
-<joint name="base_link_to_base_footprint" type="fixed">
-  <origin xyz="0 0 0" rpy="0 0 0"/>
-  <parent link="base_link"/>
-  <child link="base_footprint"/>
-</joint>
 <link name="roue_avd_1">
   <inertial>
